File: StatisSynthPcb/StatisSynthPcb.kicad_pcb (KiCad board)
At the start: 2 copper layers, 19 parts, among them J1 Conn_01x02_Pin, J2 PCM5102A, J3 Oled, SW1 SW_Push, SW2 SW_Push, SW3 SW_Push, SW4 SW_Push, SW5 SW_SPST, U3 MCP3208

Commit message: chnages to code and pcb
Parts:
- removed F1: 500ma, Fuse:Fuse_1812_4532Metric_Pad1.30x3.40mm_HandSolder
- added C1: 100microFarad, Capacitor_THT:CP_Radial_D6.3mm_P2.50mm, F.Cu at (152.8, 127.0)
- added F2: Littelfuse 02301002H, Fuse:Fuseholder_Cylinder-5x20mm_Schurter_0031_8201_Horizontal_Open, F.Cu at (149.5, 109.0)
- added J4: Conn pin for power amplifier, Connector_PinSocket_2.54mm:PinSocket_1x01_P2.54mm_Vertical, F.Cu at (176.3, 112.5)
- D1: value D_Schottky -> 1N5822; footprint Diode_SMD:D_SOD-123 -> Diode_THT:D_DO-201AD_P15.24mm_Horizontal
Routing:
- net /VSYS: track 44.5 -> 7.66 mm
- net Net-(SW5-B): track 3.78 -> 0.00 mm
- net Net-(D1-A): track 2.92 -> 0.00 mm

Commit message: pcb change
Parts:
- J4: moved to B.Cu
- moved J3 87.1 mm to (133.4, 39.0)
- moved J2 62.4 mm to (104.9, 94.5)
- moved F2 48.3 mm to (106.5, 131.0)
- moved SW5 48.2 mm to (95.0, 132.0)
- moved J1 38.7 mm to (95.5, 124.0), turned to -90 degrees
- moved U3 36.4 mm to (149.0, 85.0)
- moved RV5 34.4 mm to (113.9, 57.0)
- moved SW1 34.3 mm to (95.8, 91.0)
- moved SW2 34.3 mm to (104.4, 91.0)
- moved SW3 34.3 mm to (113.0, 91.0)
- moved SW4 34.3 mm to (121.5, 91.0)
- moved RV4 34.1 mm to (98.9, 57.0)
- moved A1 32.1 mm to (122.5, 109.0), turned to 90 degrees
- moved J4 30.2 mm to (151.0, 129.0), turned to 180 degrees
- moved RV1 26.0 mm to (98.9, 78.0)
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Routing:
- net GND: track 36.9 -> 384.1 mm, vias 0 -> 2
- net +3.3V: track 27.3 -> 228.6 mm, vias 0 -> 1
- net /SDA: track 14.1 -> 139.0 mm, vias 0 -> 1
- net /SCL: track 14.8 -> 134.8 mm
- net /VSYS: track 7.66 -> 102.2 mm, vias 0 -> 1
- net /POT4: track 0.00 -> 62.0 mm
- net /BUTTON1: track 0.00 -> 52.3 mm
- net /POT1: track 0.00 -> 50.7 mm
- net /POT5: track 0.00 -> 38.1 mm
- net /ADC_BAT: track 38.2 -> 74.0 mm, vias 0 -> 2
- net /BUTTON4: track 0.00 -> 33.1 mm
- net /POT2: track 0.00 -> 28.5 mm, vias 0 -> 2
- net /BUTTON2: track 0.00 -> 28.2 mm
- net /CLK: track 0.00 -> 24.2 mm
- net /LRCK: track 0.00 -> 17.6 mm
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
Commit message: added gerbers photos bom
Parts:
- removed SW5: SW_SPST, Button_Switch_THT:SW_DIP_SPSTx01_Slide_9.78x4.72mm_W7.62mm_P2.54mm
- R4: value 390k -> 330k
Connections:
- F2 pad 1: Net-(SW5-B) -> Net-(J1-Pin_2)
Routing:
- net Net-(J1-Pin_2): track 5.53 -> 14.6 mm
- net Net-(SW5-B): track 4.29 -> 0.00 mm
- net +3.3V: track 228.6 -> 229.3 mm
- net /SDA: track 139.0 -> 139.6 mm
Other:
- board outline added: 69 x 104.2 mm
